Commit message: Update warthog.urdf.xacro
sick_tim_571 and VLP_16 added to robot model

File: warthog_description/urdf/warthog.urdf.xacro (robot description, xacro)
@@ -375,3 +375,17 @@
   <!-- Optional for Clearpath internal softwares -->
   <xacro:include filename="$(optenv CPR_URDF_EXTRAS empty.urdf)" />
+    <!-- sick_lms5 -->
+  <xacro:include filename="$(find sick_scan)/urdf/sick_scan.urdf.xacro" />
+  <xacro:sick_tim_57x name="laser" ros_topic="scan" />
+  <joint name="sick_joint" type="fixed">
+    <origin xyz="0 0 0.6" rpy="0 0.0 0"/>
+    <parent link="base_link"/>
+    <child link="laser_mount_link"/>
+    <axis xyz="0 0.0 0.0"/>
+  </joint>
+  <!-- velodyne puck VLP_16 -->
+  <xacro:include filename="$(find velodyne_description)/urdf/VLP-16.urdf.xacro"/>
+  <xacro:VLP-16 parent="base_link" name="velodyne" topic="/velodyne_points" hz="10" lasers="16" samples="1875" collision_range="0.3" min_range="0.9" max_range="130.0" noise="0.008" min_angle="-${M_PI}" max_angle="${M_PI}" gpu="false">
+    <origin xyz="0 0 0.69" rpy="0 0 0" />
+  </xacro:VLP-16>
 </robot>

Commit message: update
generic camera added to model

File: warthog_description/urdf/warthog.urdf.xacro (robot description, xacro)
@@ -389,3 +389,8 @@
     <origin xyz="0 0 0.69" rpy="0 0 0" />
   </xacro:VLP-16>
+  <!--generic camera-->
+  <xacro:include filename="$(find warthog_description)/urdf/accessories/generic_camera.urdf.xacro" />
+  <xacro:generic_camera name="camera" parent="top_chassis_link" ros_topic="image_raw" cam_info_topic="camera_info" update_rate="30" res_x="800" res_y="600" image_format="R8G8B8" hfov="50">
+    <origin xyz="0.63 0 0.2" rpy="0 0 0"/>
+  </xacro:generic_camera>
 </robot>
